Commit message: Sensor Upgrade

File: src/my_robot/urdf/my_robot.xacro (robot description, xacro)
@@ -159,4 +159,11 @@
     <axis xyz="0 1 0" rpy="0 0 0"/>
   </joint>
+   <joint name="camera_optical_joint" type="fixed">
+    <origin xyz="0 0 0" rpy="-1.5707 0 -1.5707"/>
+    <parent link="camera_link"/>
+    <child link="camera_link_optical"/>
+  </joint>
+  <link name="camera_link_optical">
+  </link>
   <link name='hokuyo'>
     <inertial>

Commit message: Sensor Upgrade

File: src/my_robot/urdf/my_robot.xacro (robot description, xacro)
@@ -161,5 +161,5 @@
    <joint name="camera_optical_joint" type="fixed">
     <origin xyz="0 0 0" rpy="-1.5707 0 -1.5707"/>
-    <parent link="camera_link"/>
+    <parent link="camera"/>
     <child link="camera_link_optical"/>
   </joint>
